File: hardware/relay-board/relay-board.kicad_sch (KiCad schematic)
At the start: 31 parts, among them J1 ESP32-S3-ETH, J2 STOP LOOP, K1 SR4D4005, K2 SR4D4005, Q1 AO3400A, Q2 AO3400A

Commit message: docs(hardware): redraw relay board schematic to be human-readable
The first schematic connected everything with global labels and scattered
symbols: correct but unreadable (cosmetic score 32/100).

Redrawn to standard conventions: signal flow left to right, +5V/+3V3 at the
top and GND at the bottom, one dashed frame per function (J1 interface,
channel A, channel B, stop loop), wires for local connections and labels
only across frames. The SR4D4005 is now a five-unit IEC split symbol, so the
coil, NC mirror contacts and NO loop contacts are each drawn where they act,
and the four loop contacts read as a left-to-right series chain.

J1 pad order changed (power at the ends), J2 split into J2/J3 loop pads,
rail test points TP1-TP3 restored. Netlist is unchanged in substance:
check_netlist.py now matches nets by pin membership and has a built-in
--selftest with 9 injected faults. ERC clean, cosmetic score 100/100.
Parts:
- removed J2: STOP LOOP, Connector_PinHeader_2.54mm:PinHeader_1x02_P2.54mm_Vertical, symbol relay-board:Conn_01x02
- added J2: LOOP IN, Connector_PinHeader_2.54mm:PinHeader_1x01_P2.54mm_Vertical, symbol relay-board:Conn_01x01
- added J3: LOOP OUT, Connector_PinHeader_2.54mm:PinHeader_1x01_P2.54mm_Vertical, symbol relay-board:Conn_01x01
- added unit 2 of K1
- added unit 5 of K1
- added unit 3 of K1
- added unit 4 of K1
- added unit 3 of K2
- added unit 4 of K2
- added unit 2 of K2
- added unit 5 of K2
- D1, D2: Note Coil clamp (fast release). Unidirectional TVS. -> coil clamp
- J1: Note Solder wire pads (no header fitted). 1 VBUS(pin40) 2 GND 3 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 -> Solder wire pads, no header fitted. Wire to the ESP32-S3-ET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
- K1, K2: LCSC C1525104 -> (none); MPN SR4D4005 -> (none); Manufacturer TE Connectivity -> (none); Note Consigned to JLCPCB; force-guided type A -> (none)
- TP4: value GATE_A -> GATE
- TP5: value GATE_B -> GATE
- TP6: value COIL_A_N -> COIL
- TP7: value COIL_B_N -> COIL
- TP8: value MIRROR_A -> MIRROR
- TP9: value MIRROR_B -> MIRROR
Connections:
- net +3V3: now also J1.2 (Pin_2); no longer J1.7 (Pin_7)
- net GND: now also J1.7 (Pin_7), K1.11, K2.11; no longer J1.2 (Pin_2), K1.11, K2.11
- net LOOP_IN: now also J2.1 (Pin_1), K1.34; no longer K1.34
- net LOOP_MID: now also K1.44, K2.34; no longer K1.44, K2.34
- net LOOP_OUT: now also J3.1 (Pin_1), K2.44; no longer K2.44
- net COIL_A_N: no longer names the net of D1.1 (K), K1.A2, Q1.3 (D), TP6.1
- net COIL_B_N: no longer names the net of D2.1 (K), K2.A2, Q2.3 (D), TP7.1
- net GATE_A: no longer names the net of Q1.1 (G), R1.2, R3.1, TP4.1
- net GATE_B: no longer names the net of Q2.1 (G), R2.2, R4.1, TP5.1
- removed net K1_NC_LINK: K1.12, K1.22
- removed net K1_NO_LINK: K1.33, K1.43
- removed net K2_NC_LINK: K2.12, K2.22
- removed net K2_NO_LINK: K2.33, K2.43
- net MIRROR_A: no longer names the net of R5.2, R7.1, TP8.1
- net MIRROR_A: now also K1.21; no longer K1.21
- net MIRROR_B: no longer names the net of R6.2, R8.1, TP9.1
- net MIRROR_B: now also K2.21; no longer K2.21
- new net: K1.12, K1.22
- new net: K1.33, K1.43
- new net: K2.12, K2.22
- new net: K2.33, K2.43
Other:
- note added: "+5V bulk (both coils)"
- note added: "CHANNEL A (core 0): coil drive + contact mirror"
- note added: "CHANNEL B (core 1): coil drive + contact mirror"
- note added: "COIL DRIVE (fail-off: gate pulled down)"
- note added: "CONTACT MIRROR (feedback to MCU)"
- note added: "Fail-safe: de-energized = loop open. Power loss, reset, floating GPIO or a broken wire all leave both relays released. Each relay is force-guided (EN 61810-3 type A): if a NO contact welds, every NC contact of that relay stays >= 0.5 mm open. The NC mirror therefore proves the loop contacts released. Commanded 0, SNS reads 0: released, healthy. Commanded 1, SNS reads 1: pulled in, healthy. Comman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"
- note added: "HOW IT WORKS"
- note added: "J1 ESP32-S3-ETH wire pads"
- note added: "K1 coil A1-A2 (SR4D4005, 5 V, 161 mA)"
- note added: "K1: NC 21-22 and NC 11-12 in series. Closed only while released: SNS = 0 released (safe) SNS = 1 energized / weld"
- note added: "K2 coil A1-A2 (SR4D4005, 5 V, 161 mA)"
- note added: "K2: NC 21-22 and NC 11-12 in series. Closed only while released: SNS = 0 released (safe) SNS = 1 energized / weld"
- note added: "M3 holes match the 44.86 x 33.57 mm standoff pattern in machine-casing.FCStd."
- note added: "MECHANICAL"
- note added: "NO 33-34"
- note added: "NO 33-34 + NO 43-44 in series inside each relay, then K1 in series with K2: 4 gaps split the DC arc. Nothing may bridge these contacts (no TVS, snubber, LED). Fit the flyback diode / TVS at the LOAD (contactor or relay coil)."
- note added: "NO 43-44"
- note added: "PIN ESP32-S3-ETH 1 VBUS (left hdr pin 40) 2 3V3 (left hdr pin 36) 3 IO39 (right hdr pin 12) 4 IO40 (pin 11) 5 IO41 (pin 10) 6 IO42 (pin 9) 7 GND (pin 8 or 13)"
- note added: "SMAJ12A clamps the coil kick at ~20 V (fast release; a plain diode is slow)"
- note added: "STOP LOOP (dry contacts, <= 24 V DC, <= 500 mA, inductive) - drawn released"
- note added: "TEST POINTS"
- company: (none) -> Polymath Robotics
- title: (none) -> Machine relay board: dual force-guided safety relays
